File: pcb/annunciator.kicad_pcb (KiCad board)
At the start: 2 copper layers, 100 x 100 mm, 53 parts, among them J1 RPI Pico pins 1-20, J2 RPI Pico pins 21-40, J3 Display IN, Q1 2N3904, Q2 2N3904, Q3 2N3904, Q4 2N3904, Q5 2N3904, SW1 ACK, SW2 RESET, SW3 TEST, U1 74HC595, U2 74HC595

Commit message: Finish PCB work
Parts:
- added G***: LOGO, annunciator:checkm8, F.Cu at (88.8, 143.0)
- added Q6: 2N3904, Package_TO_SOT_THT:TO-92_Inline, B.Cu at (55.0, 93.1)
- added Q7: 2N3904, Package_TO_SOT_THT:TO-92_Inline, B.Cu at (55.0, 103.0)
- added Q8: 2N3904, Package_TO_SOT_THT:TO-92_Inline, B.Cu at (55.0, 111.0)
- added R24: 1k, Resistor_THT:R_Axial_DIN0207_L6.3mm_D2.5mm_P10.16mm_Horizontal, B.Cu at (114.6, 104.2)
- added R25: 1k, Resistor_THT:R_Axial_DIN0207_L6.3mm_D2.5mm_P10.16mm_Horizontal, B.Cu at (114.3, 110.5)
- added R26: 1k, Resistor_THT:R_Axial_DIN0207_L6.3mm_D2.5mm_P10.16mm_Horizontal, B.Cu at (129.0, 104.5)
- added R27: 1k, Resistor_THT:R_Axial_DIN0207_L6.3mm_D2.5mm_P10.16mm_Horizontal, B.Cu at (129.6, 110.8)
- added R28: 1k, Resistor_THT:R_Axial_DIN0207_L6.3mm_D2.5mm_P10.16mm_Horizontal, B.Cu at (132.7, 105.5)
- added R29: 1k, Resistor_THT:R_Axial_DIN0207_L6.3mm_D2.5mm_P10.16mm_Horizontal, B.Cu at (147.8, 110.5)
- moved R23 33.1 mm to (81.7, 112.5), turned to 0 degrees
- moved R22 14.7 mm to (85.8, 97.4), turned to -90 degrees
- moved D13 7.07 mm to (90.2, 106.6), turned to 90 degrees
- moved Q5 1.90 mm to (80.5, 104.4)
Connections:
- J3 pad 3: /DISP_DIN -> /DIN_5V
- J3 pad 4: /DISP_CS -> /CS_5V
- J3 pad 5: /DISP_CLK -> /CLK_5V
Routing:
- net +3V3: track 0.00 -> 223.2 mm, vias 0 -> 5
- net +5V: track 0.00 -> 203.5 mm, vias 0 -> 5
- net Net-(Q8-B): track 0.00 -> 145.7 mm, vias 0 -> 8
- net /CLK_5V: track 0.00 -> 99.0 mm, vias 0 -> 5
- net /DIN_5V: track 0.00 -> 95.6 mm, vias 0 -> 2
- net Net-(Q7-B): track 0.00 -> 90.0 mm, vias 0 -> 6
- net Net-(D13-A): track 0.00 -> 84.2 mm, vias 0 -> 2
- net /CS_5V: track 0.00 -> 82.3 mm, vias 0 -> 8
- net /SR_LATCH: track 0.00 -> 80.2 mm, vias 0 -> 6
- net /SR_CLK: track 0.00 -> 69.1 mm, vias 0 -> 4
- net Net-(Q6-B): track 0.00 -> 68.0 mm, vias 0 -> 3
- net /SR_OE: track 0.00 -> 65.8 mm, vias 0 -> 4
- net /BTN_RESET: track 0.00 -> 59.8 mm, vias 0 -> 1
- net Net-(D13-K): track 0.00 -> 59.0 mm, vias 0 -> 2
- net /BTN_ACK: track 0.00 -> 53.6 mm
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- added copper zone on B.Cu, net GND
- added copper zone on F.Cu, net GND
Other:
- board text added: "Desk Annunciator Panel Hack Club Half Life Week 4"
- board text added: "checkm8."
- board text added: "「"
- board text added: "変 わ ら な い わ か っ て ん だ よ 。"
- board text added: "頬 杖 つ い て る よ う じ ゃ"
