File: pcb/annunciator.kicad_sch (KiCad schematic)
At the start: 53 parts, among them J1 RPI Pico pins 1-20, J2 RPI Pico pins 21-40, J3 Display IN, Q1 2N3904, Q2 2N3904, Q3 2N3904, Q4 2N3904, Q5 2N3904, SW1 ACK, SW2 RESET, SW3 TEST, U1 74HC595, U2 74HC595

Commit message: Finish PCB work
Parts:
- added Q6, Q7, Q8: 2N3904, Package_TO_SOT_THT:TO-92_Inline, symbol Transistor_BJT:2N3904
- added R24, R25, R26, R27, R28, R29: 1k, Resistor_THT:R_Axial_DIN0207_L6.3mm_D2.5mm_P10.16mm_Horizontal, symbol Device:R
Connections:
- net +5V: now also R25.1, R27.1, R29.1
- net DISP_CLK: now also R28.1; no longer J3.5 (Pin_5)
- net DISP_CS: now also R26.1; no longer J3.4 (Pin_4)
- net DISP_DIN: now also R24.1; no longer J3.3 (Pin_3)
- net GND: now also Q6.1 (E), Q7.1 (E), Q8.1 (E)
- new net: Q7.2 (B), R26.2
- new net: Q8.2 (B), R28.2
- new net: Q6.2 (B), R24.2
- new net CLK_5V: J3.5 (Pin_5), Q8.3 (C), R29.2
- new net CS_5V: J3.4 (Pin_4), Q7.3 (C), R27.2
- new net DIN_5V: J3.3 (Pin_3), Q6.3 (C), R25.2
Other:
- moved on the sheet: J3
